File: protoLoad.brd (EAGLE design)
At the start: 50.8 x 50.5 mm, 37 parts, among them IC1 CP210X_USB_UART, IC2 REG1117, IC3 LM741D, IC4 LM741D, IC5 LM741D, J1 AVR_SPI_PRG_6NS, U1 ATMEGA168

Commit message: added board 3d imageand little update on brd file, placements
Parts:
- moved R5 48.3 mm to (25.4, 17.8)
- moved R7 43.0 mm to (25.4, 20.3), turned to 180 degrees
- moved R6 23.3 mm to (34.3, 39.4)
- moved C5 2.54 mm to (15.2, 10.2)
- moved R3 2.54 mm to (15.2, 12.7)
- moved D1 1.27 mm to (6.35, 33.0)
- moved IC2 1.27 mm to (6.35, 12.7)
- moved JP1 1.27 mm to (6.35, 24.1)
- moved LED1 1.27 mm to (15.2, 15.2)
Connections:
- removed net MCU_RST: U1.30
- net MCU_RXT: now also U1.30
